File: D21cpu.kicad_sch (KiCad schematic)
At the start: 11 parts, among them IC1 AVR64DD28-I_STX, J1 pad, J10 Next18, J2 pad, J3 pad

Commit message: migrated to Kicad 10
Parts:
- J1, J2, J3: footprint RTB:DummyNet-Connector -> RTB:Solder 0.8 x 0.5
Connections:
- net +3V3 renamed VDD
Changed lines of the file:
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@@
 	(title_block
 		(title "RTB D21 Next18 Decoder")
-		(date "2026-06-14")
-		(rev "0")
+		(date "2026-07-02")
+		(rev "1")
 		(company "Frank Schumacher")
 		(comment 1 "Double sided Next18")
-		(comment 2 "D21.0")
+		(comment 2 "D21.1")
 		(comment 4 "Licensed under the Apache License, Version 2")
 	)
@@
 			)
 		)
-		(property "Value" "+3V3"
-			(at 76.581 37.5158 90)
+		(property "Value" "VDD"
+			(at 76.2 36.83 90)
 			(show_name no)
 			(do_not_autoplace no)
@@
 		(property "Description" ""
 			(at 76.2 41.91 0)
+			(hide yes)
 			(show_name no)
 			(do_not_autoplace no)
@@
 		)
 		(property "Value" "GND"
-			(at 222.377 47.7012 90)
+			(at 224.028 48.514 0)
 			(show_name no)
 			(do_not_autoplace no)
@@
 			)
 		)
-		(property "Value" "+3V3"
-			(at 71.12 111.76 90)
+		(property "Value" "VDD"
+			(at 71.12 110.998 90)
 			(show_name no)
 			(do_not_autoplace no)
@@
 			)
 		)
-		(property "Value" "+3V3"
-			(at 104.14 80.01 90)
+		(property "Value" "VDD"
+			(at 103.124 80.01 90)
 			(show_name no)
 			(do_not_autoplace no)
@@
 		(property "Description" ""
 			(at 97.79 80.01 0)
+			(hide yes)
 			(show_name no)
 			(do_not_autoplace no)
@@
 		(property "Description" "AXK6F16347YG"
 			(at 203.2 93.98 0)
+			(hide yes)
 			(show_name no)
 			(do_not_autoplace no)
@@
 			)
 		)
-		(property "Footprint" "RTB:DummyNet-Connector"
+		(property "Footprint" "RTB:Solder 0.8 x 0.5"
 			(at 204.47 128.27 0)
 			(hide yes)
@@
 		(property "Description" ""
 			(at 204.47 128.27 0)
+			(hide yes)
 			(show_name no)
 			(do_not_autoplace no)
@@
 			)
 		)
-		(property "Footprint" "RTB:DummyNet-Connector"
+		(property "Footprint" "RTB:Solder 0.8 x 0.5"
 			(at 204.47 138.43 0)
 			(hide yes)
@@
 		(property "Description" ""
 			(at 204.47 138.43 0)
+			(hide yes)
 			(show_name no)
 			(do_not_autoplace no)
@@
 			)
 		)
-		(property "Footprint" "RTB:DummyNet-Connector"
+		(property "Footprint" "RTB:Solder 0.8 x 0.5"
 			(at 204.47 133.35 0)
 			(hide yes)
@@
 		(property "Description" ""
 			(at 204.47 133.35 0)
+			(hide yes)
 			(show_name no)
 			(do_not_autoplace no)
@@
 			)
 		)
-		(property "Value" "+3V3"
-			(at 194.9958 132.969 90)
+		(property "Value" "VDD"
+			(at 194.31 133.35 90)
 			(show_name no)
 			(do_not_autoplace no)
@@
 		(property "Description" ""
 			(at 199.39 133.35 0)
+			(hide yes)
 			(show_name no)
 			(do_not_autoplace no)
@@
 			)
 		)
-		(property "Value" "+3V3"
-			(at 83.82 127 90)
+		(property "Value" "VDD"
+			(at 83.312 127 90)
 			(show_name no)
 			(do_not_autoplace no)
@@
 		(property "Description" ""
 			(at 77.47 127 0)
+			(hide yes)
 			(show_name no)
 			(do_not_autoplace no)
@@
 			)
 		)
-		(property "Value" "+3V3"
-			(at 83.82 138.43 90)
+		(property "Value" "VDD"
+			(at 83.312 138.43 90)
 			(show_name no)
 			(do_not_autoplace no)
@@
 		(property "Description" ""
 			(at 77.47 138.43 0)
+			(hide yes)
 			(show_name no)
 			(do_not_autoplace no)
