File: D21rcm.kicad_sch (KiCad schematic)
At the start: 9 parts, among them Q1 BC847BDW1, Q2 BC857BDW1

Commit message: migrated to Kicad 10
Connections:
- net +3V3 renamed VDD
Changed lines of the file:
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@@
 	(title_block
 		(title "RTB D21 Next18 Decoder")
-		(date "2026-06-14")
-		(rev "0")
+		(date "2026-07-02")
+		(rev "1")
 		(company "Frank Schumacher")
 		(comment 1 "Double sided Next18")
-		(comment 2 "D21.0")
+		(comment 2 "D21.1")
 		(comment 4 "Licensed under the Apache License, Version 2")
 	)
@@
 			)
 		)
-		(property "Value" "+3V3"
+		(property "Value" "VDD"
 			(at 84.201 28.6258 0)
 			(show_name no)
@@
 		(property "Description" ""
 			(at 83.82 33.02 0)
-			(show_name no)
-			(do_not_autoplace no)
+			(hide yes)
+			(show_name no)
+			(do_not_autoplace no)
