File: D21.kicad_pcb (KiCad board)
At the start: 6 copper layers, 15.2 x 9.5 mm, 48 parts, among them IC1 AVR64DD28-I_STX, IC2 NCP730BMT500TBG, IC3 DRV8231ADSGR, J1 pad, J10 Next18, J2 pad, J3 pad, Q1 BC847BDW1, Q2 BC857BDW1, Q3 PMZB200UNEYL, Q4 PMZB200UNEYL, Q5 PMZB200UNEYL, Q6 PMZB200UNEYL

Commit message: migrated to Kicad 10
Parts:
- J1, J2, J3: footprint RTB:DummyNet-Connector -> RTB:Solder 0.8 x 0.5
- moved J1 0.10 mm to (55.7, -48.2)
- moved J3 0.09 mm to (54.5, -48.2)
- moved J2 0.09 mm to (53.2, -48.2)
Connections:
- net +3V3 renamed VDD
Other:
- board text added: "U -+"

Commit message: mod: code cleanup
Parts:
- IC2: value NCP730BMT500TBG -> NCP730BMT330TBG
Changed lines of the file:
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@@
 			)
 		)
-		(property "Value" "NCP730BMT500TBG"
+		(property "Value" "NCP730BMT330TBG"
 			(at 0 -1.95 90)
 			(layer "B.Fab")
@@
 			)
 		)
-		(property "Description" "LDO Regulator Pos 3.3V 0.15A 6-Pin WDFN EP T/R"
+		(property "Description" "-40℃~+125℃@(Tj) 1 1.8uA 150mA 195uVrms 3.3V 38V 480mV@(150mA) 80dB@(10Hz) Fixed Positive Under Voltage Lockout、Over Current Protection、Over Temperature Protection、Enable WDFN-6-EP(2x2) Voltage Regulators - Linear, Low Drop Out (LDO) Regulators ROHS"
 			(at 0 0 90)
 			(layer "F.Fab")
@@
 			)
 		)
-		(property "LCSC Part #" "C892822"
+		(property "LCSC Part #" "C892821"
 			(at 0 0 90)
 			(unlocked yes)
