File: D21pwr.kicad_sch (KiCad schematic)
At the start: 28 parts, among them IC2 NCP730BMT500TBG, IC3 DRV8231ADSGR, Q3 PMZB200UNEYL, Q4 PMZB200UNEYL, Q5 PMZB200UNEYL, Q6 PMZB200UNEYL

Commit message: migrated to Kicad 10
Parts:
- IC2: LCSC Part # (none) -> C892822
- R13: LCSC Part # C25890 -> C11702
Connections:
- net +3V3 renamed VDD
Other:
- note added: "Note: Decoder can operate at 3.3V or 5V"
- moved on the sheet: C10, C6, IC3, R13, R15, R16, R17, R18

Commit message: mod: code cleanup
Parts:
- IC2: value NCP730BMT500TBG -> NCP730BMT330TBG; LCSC Part # C892822 -> C892821
Changed lines of the file:
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@@
 			)
 		)
-		(property "Value" "NCP730BMT500TBG"
+		(property "Value" "NCP730BMT330TBG"
 			(at 177.8 33.6804 0)
 			(show_name no)
@@
 			)
 		)
-		(property "Description" "LDO Regulator Pos 3.3V 0.15A 6-Pin WDFN EP T/R"
+		(property "Description" "-40℃~+125℃@(Tj) 1 1.8uA 150mA 195uVrms 3.3V 38V 480mV@(150mA) 80dB@(10Hz) Fixed Positive Under Voltage Lockout、Over Current Protection、Over Temperature Protection、Enable WDFN-6-EP(2x2) Voltage Regulators - Linear, Low Drop Out (LDO) Regulators ROHS"
 			(at 163.83 40.64 0)
 			(hide yes)
@@
 			)
 		)
-		(property "LCSC Part #" "C892822"
+		(property "LCSC Part #" "C892821"
 			(at 195.58 38.1 0)
 			(hide yes)
